File: pilight-zero.sch (KiCad schematic (older format))
At the start: 10 parts, among them J1 GPIO partial, U1 RX-4M50RR30SF, U2 TX_433Mhz

Commit message: Replaced R2 by pot
Parts:
- R2: value 820k -> 1M; footprint Resistor_THT:R_Axial_DIN0207_L6.3mm_D2.5mm_P7.62mm_Horizontal -> Potentiometer_THT:Potentiometer_ACP_CA9-H2,5_Horizontal; symbol Device:R -> Device:R_POT_Small
Connections:
- net GND: now also R2.3; no longer R2.2
- net at U1.13 (Squelch): now also R2.2; no longer R2.1
- no-connect marks 15 -> 16
Changed lines of the file:
@@
 	4950 2100 5400 2100
 $Comp
-L Device:R R2
+L Device:R_POT_Small R2
 U 1 1 5E1DB043
-P 5350 2450
-F 0 "R2" H 5420 2496 50  0000 L CNN
-F 1 "820k" H 5420 2405 50  0000 L CNN
-F 2 "Resistor_THT:R_Axial_DIN0207_L6.3mm_D2.5mm_P7.62mm_Horizontal" V 5280 2450 50  0001 C CNN
-F 3 "~" H 5350 2450 50  0001 C CNN
-	1    5350 2450
+P 5350 2550
+F 0 "R2" H 5500 2600 50  0000 L CNN
+F 1 "1M" H 5500 2500 50  0000 L CNN
+F 2 "Potentiometer_THT:Potentiometer_ACP_CA9-H2,5_Horizontal" V 5280 2550 50  0001 C CNN
+F 3 "~" H 5350 2550 50  0001 C CNN
+	1    5350 2550
 	1    0    0    -1
 $EndComp
@@
 	1    0    0    -1
 $EndComp
-Wire Wire Line
-	5350 2600 5350 2700
-Wire Wire Line
-	5350 2300 5350 2000
-Wire Wire Line
-	5350 2000 5400 2000
 Wire Wire Line
 	5400 1600 4450 1600
@@
 	1    0    0    -1
 $EndComp
+Wire Wire Line
+	5350 2650 5350 2700
+Wire Wire Line
+	5400 2000 5350 2000
+Wire Wire Line
+	5350 2000 5350 2350
+Wire Wire Line
+	5350 2350 5450 2350
+Wire Wire Line
+	5450 2350 5450 2550
+NoConn ~ 5350 2450
 $EndSCHEMATC

Commit message: Add 3D model for trimmer
Parts:
- R2: footprint Potentiometer_THT:Potentiometer_ACP_CA9-H2,5_Horizontal -> lib:Potentiometer_ACP_CA9-H2,5_Horizontal
Changed lines of the file:
@@
 F 0 "R2" H 5500 2600 50  0000 L CNN
 F 1 "1M" H 5500 2500 50  0000 L CNN
-F 2 "Potentiometer_THT:Potentiometer_ACP_CA9-H2,5_Horizontal" V 5280 2550 50  0001 C CNN
+F 2 "lib:Potentiometer_ACP_CA9-H2,5_Horizontal" V 5280 2550 50  0001 C CNN
 F 3 "~" H 5350 2550 50  0001 C CNN
 	1    5350 2550

Commit message: Misc fixes and additions
 - Fixed pad dimensions of potentiometer
 - Added pinheader and resistors for
   - Power button
   - Power LED
   - Wifi LED
   - 433Mhz TX LED
Parts:
- added J2: Conn_02x04_Odd_Even, Connector_PinHeader_2.54mm:PinHeader_2x04_P2.54mm_Vertical, symbol Connector_Generic:Conn_02x04_Odd_Even
- added R3, R4, R5: 1k, Resistor_THT:R_Axial_DIN0207_L6.3mm_D2.5mm_P7.62mm_Horizontal, symbol Device:R
Connections:
- net GND: now also J2.1 (Pin_1), J2.3 (Pin_3), J2.5 (Pin_5), J2.7 (Pin_7)
- net GPIO14_TXD0: now also R3.1
- net GPIO17_GEN0: now also J1.11 (Pin_11), U2.3 (Data)
- net GPIO22_GEN3: now also R5.1
- net GPIO2_SDA1: now also R4.1
- net GPIO3_SCL1: now also J2.4 (Pin_4)
- new net PwrLED: J2.2 (Pin_2), R3.2
- new net TxLED: J2.8 (Pin_8), R5.2
- new net WifiLED: J2.6 (Pin_6), R4.2
- no-connect marks 16 -> 12
Changed lines of the file:
@@
 Sheet 1 1
 Title "Raspberry Pi Zero (W) uHAT for pilight"
-Date "2020-01-12"
-Rev "1.0"
+Date "2020-07-31"
+Rev "1.3"
 Comp "Fritz Elfert"
 Comment1 "This Schematic is licensed under MIT Open Source License."
@@
 Wire Wire Line
 	3950 1700 3950 1800
-Text Label 1850 1900 0    50   ~ 0
+Text Label 2300 1900 0    50   ~ 0
 GPIO2_SDA1
-Text Label 1850 2000 0    50   ~ 0
+Text Label 2300 2000 0    50   ~ 0
 GPIO3_SCL1
 Text Label 1850 2100 0    50   ~ 0
 GPIO4_GPIO_GCLK
-Text Label 1850 2300 0    50   ~ 0
+Text Label 3650 3150 0    50   ~ 0
 GPIO17_GEN0
 Text Label 1850 2400 0    50   ~ 0
@@
 	1750 2900 2800 2900
 Wire Wire Line
-	1750 2500 2800 2500
-Wire Wire Line
 	1750 2400 2800 2400
 Wire Wire Line
-	1750 2100 2800 2100
-Wire Wire Line
-	1750 2000 2800 2000
-Wire Wire Line
-	1750 1900 2800 1900
+	2050 2000 2800 2000
 Text Label 1850 2800 0    50   ~ 0
 GPIO9_SPI_MISO
 Text Label 1850 2900 0    50   ~ 0
 GPIO11_SPI_SCLK
-NoConn ~ 1750 1900
-NoConn ~ 1750 2000
-NoConn ~ 1750 2100
 NoConn ~ 1750 2400
-NoConn ~ 1750 2500
 NoConn ~ 1750 2700
 NoConn ~ 1750 2800
@@
 Wire Wire Line
 	3300 2800 4350 2800
-NoConn ~ 4350 2100
 NoConn ~ 4350 2500
 NoConn ~ 4350 2600
@@
 Wire Wire Line
 	2700 2300 2700 3150
-Wire Wire Line
-	2700 3150 5400 3150
 NoConn ~ 4350 2200
 $Comp
@@
 	5450 2350 5450 2550
 NoConn ~ 5350 2450
+$Comp
+L Connector_Generic:Conn_02x04_Odd_Even J2
+U 1 1 5F24C40E
+P 950 1800
+F 0 "J2" H 1000 2117 50  0000 C CNN
+F 1 "Conn_02x04_Odd_Even" H 1000 2026 50  0000 C CNN
+F 2 "Connector_PinHeader_2.54mm:PinHeader_2x04_P2.54mm_Vertical" H 950 1800 50  0001 C CNN
+F 3 "~" H 950 1800 50  0001 C CNN
+	1    950  1800
+	1    0    0    -1
+$EndComp
+Wire Wire Line
+	1750 2100 2800 2100
+NoConn ~ 1750 2100
+Wire Wire Line
+	2700 3150 5400 3150
+$Comp
+L power:GND #PWR0109
+U 1 1 5F28B2E2
+P 750 2250
+F 0 "#PWR0109" H 750 2000 50  0001 C CNN
+F 1 "GND" H 755 2077 50  0000 C CNN
+F 2 "" H 750 2250 50  0001 C CNN
+F 3 "" H 750 2250 50  0001 C CNN
+	1    750  2250
+	1    0    0    -1
+$EndComp
+Wire Wire Line
+	750  1700 750  1800
+Connection ~ 750  1800
+Wire Wire Line
+	750  1800 750  1900
+Connection ~ 750  1900
+Wire Wire Line
+	750  1900 750  2000
+Connection ~ 750  2000
+Wire Wire Line
+	750  2000 750  2250
+Wire Wire Line
+	2050 2000 2050 1800
+Wire Wire Line
+	2050 1800 1250 1800
+$Comp
+L Device:R R3
+U 1 1 5F2B5902
+P 4350 1850
+F 0 "R3" V 4143 1850 50  0000 C CNN
+F 1 "1k" V 4234 1850 50  0000 C CNN
+F 2 "Resistor_THT:R_Axial_DIN0207_L6.3mm_D2.5mm_P7.62mm_Horizontal" V 4280 1850 50  0001 C CNN
+F 3 "~" H 4350 1850 50  0001 C CNN
+	1    4350 1850
+	-1   0    0    1
+$EndComp
+Wire Wire Line
+	4350 2000 4350 2100
+Text Label 1300 1700 0    50   ~ 0
+PwrLED
+Text Label 1300 1800 0    50   ~ 0
+PwrButton
+Wire Wire Line
+	1250 1700 4350 1700
+Text Label 1300 1900 0    50   ~ 0
+WifiLED
+Wire Wire Line
+	1600 2000 1250 2000
+Wire Wire Line
+	1600 2500 2800 2500
+Text Label 1300 2000 0    50   ~ 0
+TxLED
+$Comp
+L Device:R R4
+U 1 1 5F312684
+P 1850 1900
+F 0 "R4" V 1643 1900 50  0000 C CNN
+F 1 "1k" V 1734 1900 50  0000 C CNN
+F 2 "Resistor_THT:R_Axial_DIN0207_L6.3mm_D2.5mm_P7.62mm_Horizontal" V 1780 1900 50  0001 C CNN
+F 3 "~" H 1850 1900 50  0001 C CNN
+	1    1850 1900
+	0    1    1    0
+$EndComp
+Wire Wire Line
+	2000 1900 2800 1900
+Wire Wire Line
+	1700 1900 1250 1900
+$Comp
+L Device:R R5
+U 1 1 5F3354AF
+P 1600 2250
+F 0 "R5" V 1393 2250 50  0000 C CNN
+F 1 "1k" V 1484 2250 50  0000 C CNN
+F 2 "Resistor_THT:R_Axial_DIN0207_L6.3mm_D2.5mm_P7.62mm_Horizontal" V 1530 2250 50  0001 C CNN
+F 3 "~" H 1600 2250 50  0001 C CNN
+	1    1600 2250
+	-1   0    0    1
+$EndComp
+Wire Wire Line
+	1600 2500 1600 2400
+Wire Wire Line
+	1600 2100 1600 2000
 $EndSCHEMATC

Commit message: Updated misc 3d models
Parts:
- U2: footprint Connector_PinHeader_2.54mm:PinHeader_1x03_P2.54mm_Vertical -> lib:TX-433Mhz
Other:
- note added: "Externally wired"
- note added: "PwrButton"
- note added: "PwrLED"
- note added: "TxLED"
- note added: "WifiLED"
Changed lines of the file:
@@
 F 0 "U2" H 5778 3401 50  0000 L CNN
 F 1 "TX_433Mhz" H 5778 3310 50  0000 L CNN
-F 2 "Connector_PinHeader_2.54mm:PinHeader_1x03_P2.54mm_Vertical" H 5600 3300 50  0001 C CNN
+F 2 "lib:TX-433Mhz" H 5600 3300 50  0001 C CNN
 F 3 "" H 5600 3300 50  0001 C CNN
 	1    5600 3300
@@
 Wire Wire Line
 	1600 2100 1600 2000
+$Comp
+L Connector_Generic:Conn_02x04_Odd_Even #J2
+U 1 1 5F250DB8
+P 2950 5350
+F 0 "#J2" H 3000 5667 50  0000 C CNN
+F 1 "Conn_02x04_Odd_Even" H 3000 5576 50  0000 C CNN
+F 2 "" H 2950 5350 50  0001 C CNN
+F 3 "~" H 2950 5350 50  0001 C CNN
+	1    2950 5350
+	1    0    0    -1
+$EndComp
+$Comp
+L Device:LED #D1
+U 1 1 5F25BDFB
+P 3000 4800
+F 0 "#D1" H 2993 5017 50  0000 C CNN
+F 1 "LED" H 2993 4926 50  0000 C CNN
+F 2 "" H 3000 4800 50  0001 C CNN
+F 3 "~" H 3000 4800 50  0001 C CNN
+	1    3000 4800
+	1    0    0    -1
+$EndComp
+$Comp
+L Device:LED #D3
+U 1 1 5F27004E
+P 3000 5900
+F 0 "#D3" H 2993 6117 50  0000 C CNN
+F 1 "LED" H 2993 6026 50  0000 C CNN
+F 2 "" H 3000 5900 50  0001 C CNN
+F 3 "~" H 3000 5900 50  0001 C CNN
+	1    3000 5900
+	1    0    0    -1
+$EndComp
+$Comp
+L Device:LED #D2
+U 1 1 5F270844
+P 3000 6250
+F 0 "#D2" H 2993 6467 50  0000 C CNN
+F 1 "LED" H 2993 6376 50  0000 C CNN
+F 2 "" H 3000 6250 50  0001 C CNN
+F 3 "~" H 3000 6250 50  0001 C CNN
+	1    3000 6250
+	1    0    0    -1
+$EndComp
+$Comp
+L Switch:SW_Push #SW1
+U 1 1 5F2717D6
+P 3000 4450
+F 0 "#SW1" H 3000 4735 50  0000 C CNN
+F 1 "SW_Push" H 3000 4644 50  0000 C CNN
+F 2 "" H 3000 4650 50  0001 C CNN
+F 3 "~" H 3000 4650 50  0001 C CNN
+	1    3000 4450
+	1    0    0    -1
+$EndComp
+Wire Wire Line
+	3150 4800 3450 4800
+Wire Wire Line
+	3450 4800 3450 5250
+Wire Wire Line
+	3450 5250 3250 5250
+Wire Wire Line
+	3200 4450 3550 4450
+Wire Wire Line
+	3550 4450 3550 5350
+Wire Wire Line
+	3550 5350 3250 5350
+Wire Wire Line
+	2850 4800 2500 4800
+Wire Wire Line
+	2500 4800 2500 5250
+Wire Wire Line
+	2500 5250 2750 5250
+Wire Wire Line
+	2800 4450 2400 4450
+Wire Wire Line
+	2400 4450 2400 5350
+Wire Wire Line
+	2400 5350 2750 5350
+Wire Wire Line
+	3250 5550 3450 5550
+Wire Wire Line
+	3450 5550 3450 5900
+Wire Wire Line
+	3450 5900 3150 5900
+Wire Wire Line
+	2750 5550 2500 5550
+Wire Wire Line
+	2500 5550 2500 5900
+Wire Wire Line
+	2500 5900 2850 5900
+Wire Wire Line
+	3250 5450 3550 5450
+Wire Wire Line
+	3550 5450 3550 6250
+Wire Wire Line
+	3550 6250 3150 6250
+Wire Wire Line
+	2750 5450 2400 5450
+Wire Wire Line
+	2400 5450 2400 6250
+Wire Wire Line
+	2400 6250 2850 6250
+Wire Notes Line
+	1750 3900 1750 6450
+Wire Notes Line
+	1750 6450 4000 6450
+Wire Notes Line
+	4000 6450 4000 3900
+Wire Notes Line
+	4000 3900 1750 3900
+Text Notes 1850 4050 0    50   ~ 0
+Externally wired
+Text Notes 1850 4500 0    50   ~ 0
+PwrButton
+Text Notes 1850 4850 0    50   ~ 0
+PwrLED
+Text Notes 1850 6300 0    50   ~ 0
+WifiLED
+Text Notes 1850 5950 0    50   ~ 0
+TxLED
+Wire Notes Line
+	3000 5400 1000 5400
+Wire Notes Line
+	1000 5400 1000 1850
 $EndSCHEMATC

Commit message: Changed WifiLED output to GPIO27
Connections:
- net GPIO27_GEN2: now also R4.1
- net GPIO2_SDA1: no longer R4.1
Other:
- moved on the sheet: R4, R5
Changed lines of the file:
@@
 Sheet 1 1
 Title "Raspberry Pi Zero (W) uHAT for pilight"
-Date "2020-07-31"
-Rev "1.3"
+Date "2020-08-02"
+Rev "1.4"
 Comp "Fritz Elfert"
 Comment1 "This Schematic is licensed under MIT Open Source License."
@@
 	1750 2900 2800 2900
 Wire Wire Line
-	1750 2400 2800 2400
-Wire Wire Line
 	2050 2000 2800 2000
 Text Label 1850 2800 0    50   ~ 0
@@
 Text Label 1850 2900 0    50   ~ 0
 GPIO11_SPI_SCLK
-NoConn ~ 1750 2400
 NoConn ~ 1750 2700
 NoConn ~ 1750 2800
@@
 WifiLED
 Wire Wire Line
-	1600 2000 1250 2000
-Wire Wire Line
-	1600 2500 2800 2500
+	1550 2000 1250 2000
+Wire Wire Line
+	1550 2500 2800 2500
 Text Label 1300 2000 0    50   ~ 0
 TxLED
@@
 L Device:R R4
 U 1 1 5F312684
-P 1850 1900
-F 0 "R4" V 1643 1900 50  0000 C CNN
-F 1 "1k" V 1734 1900 50  0000 C CNN
-F 2 "Resistor_THT:R_Axial_DIN0207_L6.3mm_D2.5mm_P7.62mm_Horizontal" V 1780 1900 50  0001 C CNN
-F 3 "~" H 1850 1900 50  0001 C CNN
-	1    1850 1900
-	0    1    1    0
-$EndComp
-Wire Wire Line
-	2000 1900 2800 1900
-Wire Wire Line
-	1700 1900 1250 1900
+P 1650 2050
+F 0 "R4" V 1443 2050 50  0000 C CNN
+F 1 "1k" V 1534 2050 50  0000 C CNN
+F 2 "Resistor_THT:R_Axial_DIN0207_L6.3mm_D2.5mm_P7.62mm_Horizontal" V 1580 2050 50  0001 C CNN
+F 3 "~" H 1650 2050 50  0001 C CNN
+	1    1650 2050
+	-1   0    0    1
+$EndComp
+Wire Wire Line
+	1750 1900 2800 1900
 $Comp
 L Device:R R5
 U 1 1 5F3354AF
-P 1600 2250
-F 0 "R5" V 1393 2250 50  0000 C CNN
-F 1 "1k" V 1484 2250 50  0000 C CNN
-F 2 "Resistor_THT:R_Axial_DIN0207_L6.3mm_D2.5mm_P7.62mm_Horizontal" V 1530 2250 50  0001 C CNN
-F 3 "~" H 1600 2250 50  0001 C CNN
-	1    1600 2250
+P 1550 2250
+F 0 "R5" V 1343 2250 50  0000 C CNN
+F 1 "1k" V 1434 2250 50  0000 C CNN
+F 2 "Resistor_THT:R_Axial_DIN0207_L6.3mm_D2.5mm_P7.62mm_Horizontal" V 1480 2250 50  0001 C CNN
+F 3 "~" H 1550 2250 50  0001 C CNN
+	1    1550 2250
 	-1   0    0    1
 $EndComp
 Wire Wire Line
-	1600 2500 1600 2400
-Wire Wire Line
-	1600 2100 1600 2000
+	1550 2500 1550 2400
+Wire Wire Line
+	1550 2100 1550 2000
 $Comp
 L Connector_Generic:Conn_02x04_Odd_Even #J2
@@
 Wire Notes Line
 	1000 5400 1000 1850
+Wire Wire Line
+	1650 1900 1250 1900
+NoConn ~ 1750 1900
+Wire Wire Line
+	1650 2200 1650 2400
+Wire Wire Line
+	1650 2400 2800 2400
 $EndSCHEMATC
